File: Rev A/SurgicalLightBoostConverterModule.kicad_pcb (KiCad board)
At the start: 2 copper layers, 0 parts

Commit message: PCB? :(
Parts:
- added 1IN+: 1IN+, TestPoint:TestPoint_Pad_D2.0mm, F.Cu at (96.5, 104.0)
- added 1IN-: 1IN-, TestPoint:TestPoint_Pad_D2.0mm, F.Cu at (92.0, 104.0)
- added 24V: 24V, TestPoint:TestPoint_Pad_D2.0mm, F.Cu at (150.0, 38.5)
- added 2IN+: 2IN+, TestPoint:TestPoint_Pad_D2.0mm, F.Cu at (108.5, 104.0)
- added 2IN-: 2IN-, TestPoint:TestPoint_Pad_D2.0mm, F.Cu at (113.0, 104.0)
- added 5V: 5V, TestPoint:TestPoint_Pad_D2.0mm, F.Cu at (74.5, 77.5)
- added C1: 0.1uF, Capacitor_SMD:C_0805_2012Metric, F.Cu at (49.6, 93.0)
- added C10: 1uF, Capacitor_SMD:C_0805_2012Metric, F.Cu at (147.1, 79.2)
- added C11: 0.1uF, Capacitor_SMD:C_0805_2012Metric, F.Cu at (144.6, 79.2)
- added C2: 470uF, Capacitor_THT:CP_Radial_D12.5mm_P5.00mm, F.Cu at (47.2, 65.0)
- added C3: 470uF, Capacitor_THT:CP_Radial_D12.5mm_P5.00mm, F.Cu at (47.2, 81.5)
- added C4: 220uF, Capacitor_THT:CP_Radial_D10.0mm_P5.00mm, F.Cu at (106.0, 29.5)
- added C5: 220uF, Capacitor_THT:CP_Radial_D10.0mm_P5.00mm, F.Cu at (106.0, 44.0)
- added C6: 0.1uF, Capacitor_SMD:C_0805_2012Metric, F.Cu at (108.5, 54.0)
- added C7: 1uF, Capacitor_SMD:C_0805_2012Metric, F.Cu at (115.3, 84.5)
- added C8: 0.1uF, Capacitor_SMD:C_0805_2012Metric, F.Cu at (112.8, 84.5)
- added C9: 1nF, Capacitor_SMD:C_0805_2012Metric, F.Cu at (94.8, 88.5)
- added D1: PMEG045V150EPD, Package_TO_SOT_SMD:Nexperia_CFP15_SOT-1289, F.Cu at (81.8, 27.0)
- added D2: LED Green, LED_SMD:LED_0805_2012Metric, F.Cu at (133.3, 44.0)
- added D3: LED Green, LED_SMD:LED_0805_2012Metric, F.Cu at (39.4, 68.9)
- added D4: LED Green, LED_SMD:LED_0805_2012Metric, F.Cu at (117.7, 70.5)
- added D5: LED Red, LED_SMD:LED_0805_2012Metric, F.Cu at (64.9, 68.0)
- added D6: PMEG045V150EPD, Package_TO_SOT_SMD:Nexperia_CFP15_SOT-1289, F.Cu at (67.9, 88.5)
- added DTC: DTC, TestPoint:TestPoint_Pad_D2.0mm, F.Cu at (102.5, 104.0)
- added F1: 12A, Fuse:Fuse_1206_3216Metric_Pad1.42x1.75mm_HandSolder, F.Cu at (116.4, 24.5)
- added H1: M3 Hole, MountingHole:MountingHole_3.2mm_M3_Pad_TopBottom, F.Cu at (30.0, 100.0)
- added H2: M3 Hole, MountingHole:MountingHole_3.2mm_M3_Pad_TopBottom, F.Cu at (150.0, 100.0)
- added H3: M3 Hole, MountingHole:MountingHole_3.2mm_M3_Pad_TopBottom, F.Cu at (150.0, 30.0)
- added H4: M3 Hole, MountingHole:MountingHole_3.2mm_M3_Pad_TopBottom, F.Cu at (30.0, 30.0)
- added L1: 68uH 11.4A, Inductor_THT:L_Radial_D29.8mm_P29.30mm_Murata_1400series, F.Cu at (40.7, 40.0)
- added PWM: PWM, TestPoint:TestPoint_Pad_D2.0mm, F.Cu at (118.5, 95.5)
- added Q1: IRLZ44N, Package_TO_SOT_THT:TO-220-3_Vertical, F.Cu at (89.5, 42.6)
- added Q2: IRLZ44N, Package_TO_SOT_THT:TO-220-3_Vertical, F.Cu at (89.5, 57.0)
- added Q3: BC337, Package_TO_SOT_THT:TO-92_Inline, F.Cu at (98.5, 68.0)
- added Q4: BC327, Package_TO_SOT_THT:TO-92_Inline, F.Cu at (106.8, 68.0)
- added Q5: BC327, Package_TO_SOT_THT:TO-92_Inline, F.Cu at (79.1, 82.0)
- added R1: 0R1, Resistor_SMD:R_2512_6332Metric, F.Cu at (125.3, 26.5)
- added R10: 9.1K, Resistor_SMD:R_0805_2012Metric, F.Cu at (73.0, 68.5)
- added R11: 1K, Resistor_SMD:R_0805_2012Metric, F.Cu at (95.4, 78.0)
- added R12: 1K, Resistor_SMD:R_0805_2012Metric, F.Cu at (95.4, 74.5)
- added R13: 10K, Resistor_SMD:R_0805_2012Metric, F.Cu at (88.4, 80.5)
- added R14: 100K, Resistor_SMD:R_0805_2012Metric, F.Cu at (95.4, 80.5)
- added R15: 1K, Resistor_SMD:R_0805_2012Metric, F.Cu at (73.0, 71.0)
- added R16: 2K2, Resistor_SMD:R_0805_2012Metric, F.Cu at (90.5, 86.0)
- added R17: 3K9, Resistor_SMD:R_0805_2012Metric, F.Cu at (94.8, 91.0)
- added R18: 10K, Resistor_SMD:R_0805_2012Metric, F.Cu at (125.6, 77.7)
- added R19: 10K, Resistor_SMD:R_0805_2012Metric, F.Cu at (117.0, 77.4)
- added R2: 0R1, Resistor_SMD:R_2512_6332Metric, F.Cu at (125.3, 33.5)
- added R20: 1K, Resistor_SMD:R_0805_2012Metric, F.Cu at (125.6, 83.2)
- added R21: 10K, Resistor_SMD:R_0805_2012Metric, F.Cu at (113.0, 77.4)
- added R22: 1K, Resistor_SMD:R_0805_2012Metric, F.Cu at (137.1, 71.5)
- added R23: 10K, Resistor_SMD:R_0805_2012Metric, F.Cu at (125.6, 80.5)
- added R24: 10K, Resistor_SMD:R_0805_2012Metric, F.Cu at (124.4, 68.5)
- added R3: 2K, Resistor_SMD:R_0805_2012Metric, F.Cu at (133.3, 41.4)
- added R4: 1K, Resistor_SMD:R_0805_2012Metric, F.Cu at (39.4, 65.5)
- added R5: 10, Resistor_SMD:R_0805_2012Metric, F.Cu at (101.6, 61.0)
- added R6: 330, Resistor_SMD:R_0805_2012Metric, F.Cu at (112.9, 70.5)
- added R7: 2K, Resistor_SMD:R_0805_2012Metric, F.Cu at (64.9, 65.2)
- added R8: 10K, Resistor_SMD:R_0805_2012Metric, F.Cu at (88.4, 78.0)
- added R9: 10K, Resistor_SMD:R_0805_2012Metric, F.Cu at (79.9, 77.5)
- added RV1: 10K, Connector_PinHeader_2.54mm:PinHeader_1x03_P2.54mm_Vertical, F.Cu at (82.4, 69.5)
- added RV2: 10K, Connector_PinHeader_2.54mm:PinHeader_1x03_P2.54mm_Vertical, F.Cu at (133.9, 68.5)
- added U1: TL494, Package_DIP:DIP-16_W7.62mm, F.Cu at (100.7, 75.5)
- added U2: TL431D, Package_SO:SOIC-8_3.9x4.9mm_P1.27mm, F.Cu at (67.0, 80.0)
- added U3: LM358, Package_DIP:DIP-8_W7.62mm_Socket, F.Cu at (131.3, 77.9)
Routing:
- net /CS+: track 0.00 -> 80.9 mm, vias 0 -> 2
- net +5V: track 0.00 -> 71.8 mm, vias 0 -> 2
- net Net-(Q1-D): track 0.00 -> 71.3 mm
- net GND: track 0.00 -> 68.4 mm, vias 0 -> 12
- net /2IN+: track 0.00 -> 62.5 mm, vias 0 -> 3
- net Net-(D1-K): track 0.00 -> 61.8 mm
- net BoostConverterSwitch: track 0.00 -> 55.5 mm, vias 0 -> 2
- net /1IN+: track 0.00 -> 49.1 mm, vias 0 -> 2
- net /DTC: track 0.00 -> 44.5 mm, vias 0 -> 2
- net /2IN-: track 0.00 -> 38.4 mm, vias 0 -> 2
- net /1IN-: track 0.00 -> 32.2 mm, vias 0 -> 2
- net Net-(Q1-G): track 0.00 -> 27.2 mm
- net Net-(D5-K): track 0.00 -> 25.1 mm
- net Net-(Q5-B): track 0.00 -> 19.5 mm
- net Net-(U3A-+): track 0.00 -> 18.9 mm, vias 0 -> 2
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- added copper zone on F.Cu, net +12V
- added copper zone on F.Cu, net +24V
- added copper zone on B.Cu, net GND
Other:
- board outline added: 140 x 90 mm
