File: Rev A/SurgicalLightBoostConverterModule.kicad_pcb (KiCad board)
At the start: 2 copper layers, 140 x 90 mm, 65 parts, among them Q1 IRLZ44N, Q2 IRLZ44N, Q3 BC337, Q4 BC327, Q5 BC327, U1 TL494, U2 TL431D, U3 LM358

Commit message: added michael's changes
Parts:
- removed PWM: PWM, TestPoint:TestPoint_Pad_D2.0mm
- removed the R2 at (125.3, 33.5)
- added C10: 0.1uF, Capacitor_SMD:C_0805_2012Metric, F.Cu at (74.0, 34.0)
- added C7: 0.1uF, Capacitor_SMD:C_0805_2012Metric, F.Cu at (53.0, 61.0)
- added C8: 0.1uF, Capacitor_SMD:C_0805_2012Metric, F.Cu at (70.0, 30.5)
- added C9: 0.1uF, Capacitor_SMD:C_0805_2012Metric, F.Cu at (70.0, 38.0)
- added D2: PMEG045V150EPD, Package_TO_SOT_SMD:Nexperia_CFP15_SOT-1289, F.Cu at (100.4, 27.1)
- added D5: PMEG045V150EPD, Package_TO_SOT_SMD:Nexperia_CFP15_SOT-1289, F.Cu at (106.9, 27.1)
- added D6: PMEG045V150EPD, Package_TO_SOT_SMD:Nexperia_CFP15_SOT-1289, F.Cu at (113.5, 27.1)
- added J1: 2x7 P2.54mm, Connector_PinHeader_2.54mm:PinHeader_2x07_P2.54mm_Vertical, F.Cu at (115.5, 105.7)
- added Q5: IRLZ44N, Package_TO_SOT_THT:TO-220-3_Vertical, F.Cu at (108.5, 39.0)
- added Q6: IRLZ44N, Package_TO_SOT_THT:TO-220-3_Vertical, F.Cu at (128.5, 39.0)
- added Q7: BC327, Package_TO_SOT_THT:TO-92_Inline, F.Cu at (91.0, 58.5)
- added Q8: BC327, Package_TO_SOT_THT:TO-92_Inline, F.Cu at (111.0, 58.5)
- added Q9: BC327, Package_TO_SOT_THT:TO-92_Inline, F.Cu at (131.0, 58.5)
- added R4: 10, Resistor_SMD:R_0805_2012Metric, F.Cu at (88.5, 44.1)
- added R6: 10, Resistor_SMD:R_0805_2012Metric, F.Cu at (128.5, 44.0)
- added TP1: LMount1, TestPoint:TestPoint_Loop_D2.54mm_Drill1.5mm_Beaded, F.Cu at (30.5, 23.5)
- added TP11: CS+, TestPoint:TestPoint_Loop_D2.54mm_Drill1.5mm_Beaded, F.Cu at (138.5, 60.0)
- added TP13: CS-, TestPoint:TestPoint_Loop_D2.54mm_Drill1.5mm_Beaded, F.Cu at (138.5, 66.5)
- added TP2: LMount2, TestPoint:TestPoint_Loop_D2.54mm_Drill1.5mm_Beaded, F.Cu at (69.5, 24.5)
- added TP3: LMount4, TestPoint:TestPoint_Loop_D2.54mm_Drill1.5mm_Beaded, F.Cu at (69.0, 57.5)
- added TP4: LMount3, TestPoint:TestPoint_Loop_D2.54mm_Drill1.5mm_Beaded, F.Cu at (31.0, 58.0)
- added TP9: PWM, TestPoint:TestPoint_Loop_D2.54mm_Drill1.5mm_Beaded, F.Cu at (118.5, 95.5)
- F1: footprint Fuse:Fuse_1206_3216Metric_Pad1.42x1.75mm_HandSolder -> Fuse:Fuseholder_Clip-6.3x32mm_Littelfuse_102071_Inline_P34.70x7.60mm_D2.00mm_Horizontal
- Q1, Q2: value IRLZ44N -> BC337; footprint Package_TO_SOT_THT:TO-220-3_Vertical -> Package_TO_SOT_THT:TO-92_Inline
- Q4: value BC327 -> IRLZ44N; footprint Package_TO_SOT_THT:TO-92_Inline -> Package_TO_SOT_THT:TO-220-3_Vertical
- R1: value 0R1 -> 5mR
- R19: renamed from R18; value 10K -> 100K
- R24: renamed from R23; value 10K -> 100K
- TP10: renamed from DTC; footprint TestPoint:TestPoint_Pad_D2.0mm -> TestPoint:TestPoint_Loop_D2.54mm_Drill1.5mm_Beaded
- TP12: renamed from 2IN-; footprint TestPoint:TestPoint_Pad_D2.0mm -> TestPoint:TestPoint_Loop_D2.54mm_Drill1.5mm_Beaded
- TP14: renamed from 2IN+; footprint TestPoint:TestPoint_Pad_D2.0mm -> TestPoint:TestPoint_Loop_D2.54mm_Drill1.5mm_Beaded
- TP5: renamed from 24V; footprint TestPoint:TestPoint_Pad_D2.0mm -> TestPoint:TestPoint_Loop_D2.54mm_Drill1.5mm_Beaded
- TP6: renamed from 5V; footprint TestPoint:TestPoint_Pad_D2.0mm -> TestPoint:TestPoint_Loop_D2.54mm_Drill1.5mm_Beaded
- TP7: renamed from 1IN-; footprint TestPoint:TestPoint_Pad_D2.0mm -> TestPoint:TestPoint_Loop_D2.54mm_Drill1.5mm_Beaded
- TP8: renamed from 1IN+; footprint TestPoint:TestPoint_Pad_D2.0mm -> TestPoint:TestPoint_Loop_D2.54mm_Drill1.5mm_Beaded
- U2: footprint Package_SO:SOIC-8_3.9x4.9mm_P1.27mm -> Package_DIP:DIP-8_W7.62mm_Socket
- moved C6 62.4 mm to (46.5, 61.0)
- moved F1 55.1 mm to (152.5, 66.1), turned to 90 degrees
- moved R1 41.9 mm to (145.0, 63.5), turned to -90 degrees
- moved Q3 36.9 mm to (131.0, 50.5), turned to 180 degrees
- moved R3 35.7 mm to (24.5, 33.1)
- moved D4 35.7 mm to (24.5, 36.5)
- moved Q4 34.3 mm to (88.5, 39.0), turned to 0 degrees
- moved C5 33.6 mm to (39.5, 61.0)
- moved C3 31.6 mm to (74.5, 26.9)
- moved C4 31.2 mm to (75.0, 40.9)
- moved TP5 29.1 mm to (124.0, 25.5)
- moved Q2 22.4 mm to (111.0, 50.5)
- moved R5 18.3 mm to (108.5, 44.1), turned to 90 degrees
- moved D3 13.7 mm to (146.0, 38.9), turned to -90 degrees
- moved R2 12.8 mm to (146.0, 43.4), turned to 90 degrees
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- renumbered C2 to C1, C7 to C11, C8 to C12, C9 to C13, C10 to C14, C11 to C15, C3 to C2, C4 to C3, C5 to C4, C1 to C5, D2 to D3, D3 to D4, D4 to D7, D5 to D8, D6 to D9, H3 to H1, H4 to H2, H1 to H3, H2 to H4, Q5 to Q10, R9 to R10, R10 to R11, R11 to R12, R12 to R13, R13 to R14, R14 to R15, R15 to R16, R16 to R17, R17 to R18, R3 to R2, R19 to R20, R20 to R21, R21 to R22, R22 to R23, R24 to R25, R4 to R3, R6 to R7, R7 to R8, R8 to R9
Connections:
- C3 pad 1: Net-(D1-K) -> /CS+
- C4 pad 1: Net-(D1-K) -> /CS+
- C6 pad 1: Net-(D1-K) -> +12V
- D1 pad 1: Net-(Q1-D) -> /VSwitch
- D1 pad 2: Net-(Q1-D) -> /VSwitch
- D1 pad 3: Net-(D1-K) -> /CS+
- F1 pad 1: Net-(D1-K) -> /CS-
- F1 pad 2: /CS+ -> +24V
- L1 pad 2: Net-(Q1-D) -> /VSwitch
- Q1 pad 1: Net-(Q1-G) -> /VSwitch
- Q1 pad 2: Net-(Q1-D) -> BoostConverterSwitch
- Q1 pad 3: GND -> Net-(Q1-E)
- Q2 pad 1: Net-(Q1-G) -> /VSwitch
- Q2 pad 2: Net-(Q1-D) -> BoostConverterSwitch
- Q2 pad 3: GND -> Net-(Q2-E)
- Q3 pad 1: Net-(Q1-D) -> /VSwitch
- Q4 pad 1: GND -> Net-(Q4-G)
- Q4 pad 2: BoostConverterSwitch -> /VSwitch
- Q4 pad 3: Net-(Q3-E) -> GND
- R1 pad 2: +24V -> /CS-
- R11 pad 1: +24V -> /CS+
- R2 pad 1: /CS+ -> /CS-
- R23 pad 1: +24V -> /CS-
- R5 pad 1: Net-(Q1-G) -> Net-(Q2-E)
- R5 pad 2: Net-(Q3-E) -> Net-(Q5-G)
- R8 pad 1: +24V -> /CS+
- RV1 pad 1: +24V -> /CS+
- RV1 pad 2: +24V -> /CS+
- TP5 pad 1: +24V -> /CS+
Routing:
- net BoostConverterSwitch: track 55.5 -> 129.5 mm
- net Net-(Q1-D): track 71.3 -> 0.00 mm
- net Net-(D1-K): track 61.8 -> 0.00 mm
- net /DTC: track 44.5 -> 87.5 mm, vias 2 -> 4
- net /1IN-: track 32.2 -> 64.6 mm, vias 2 -> 3
- net /CS+: track 80.9 -> 112.6 mm, vias 2 -> 3
- net Net-(Q1-G): track 27.2 -> 0.00 mm
- net /2IN-: track 38.4 -> 53.2 mm, vias 2 -> 3
- net Net-(Q2-E): track 0.00 -> 13.5 mm
- net Net-(Q1-E): track 0.00 -> 13.5 mm
- net /CS-: track 0.00 -> 13.5 mm
- net Net-(D8-K): track 25.1 -> 38.4 mm
- net /1IN+: track 49.1 -> 54.8 mm
- net Net-(Q4-G): track 0.00 -> 4.29 mm
- net Net-(Q5-G): track 0.00 -> 4.17 mm
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- added copper zone on F.Cu, net /CS+
- added copper zone on F.Cu, net /CS-
- added copper zone on F.Cu, net /VSwitch
Other:
- outline, holes or cut-outs redrawn
- board text added: "Robust Surgical Lighting - Boost Converter Module Rev A Mar 2024 ML/MIT 2.750"
